File: test_board2.sch (KiCad schematic (older format))
At the start: 77 parts, among them U1 SM220, U2 AS1116

Commit message: After 1st design review
Parts:
- removed D10, D11, D12, D13, D14, D15, D16, D17, D18, D19, D2, D20, D21, D22, D23, D24, D25, D26, D27, D28, D29, D3, D30, D31, D32, D33, D34, D35, D36, D37, D38, D39, D4, D40, D41, D42, D43, D44, D45, D46, D47, D48, D49, D5, D50, D51, D52, D53, D54, D55, D56, D57, D58, D59, D6, D60, D61, D62, D63, D64, D7, D8, D9: LED, LEDs:LED-0603, symbol LED
- removed P?: USB_B, symbol USB_B
- removed R1: 12k, Resistors_SMD:R_0603_HandSoldering, symbol R
- removed U2: AS1116, Synapse:QSOP-24, symbol AS1116
- added BT1, BT2: 1.5V, Synapse:BATT_2466, symbol Battery
- added C10, C12, C20: 0.1uF, Capacitors_SMD:C_0603, symbol C
- added C11, C15, C9: 4.7uF, Capacitors_SMD:C_0603, symbol C
- added C2, C21: 100nF, Capacitors_SMD:C_0603, symbol C
- added C22, C23, C7, C8: 22uF, Capacitors_SMD:C_0603, symbol C
- added C3: 10uF, Capacitors_SMD:C_0603, symbol C
- added C4: 10nF, Capacitors_SMD:C_0603, symbol C_Small
- added C5, C6: 47pF, Capacitors_SMD:C_0603, symbol C_Small
- added P1: MicroB, Synapse:USBmicroB, symbol USB_OTG
- added P2, P3: CONN_01X08, Pin_Headers:Pin_Header_Straight_1x08, symbol CONN_01X08
- added P4: CONN_01X10, Pin_Headers:Pin_Header_Straight_1x10, symbol CONN_01X10
- added P5: CONN_01X06, Pin_Headers:Pin_Header_Straight_1x06, symbol CONN_01X06
- added P6: CONN_02X03, Pin_Headers:Pin_Header_Straight_2x03, symbol CONN_02X03
- added Q1: ZXMN2F30FHCT-ND, TO_SOT_Packages_SMD:SOT-23, symbol Q_NMOS_GSD
- added Q2: Si2305DS, TO_SOT_Packages_SMD:SOT-23, symbol Q_PMOS_GSD
- added R12: 100k, Resistors_SMD:R_0603, symbol R_Small
- added R13: 39k, Resistors_SMD:R_0603, symbol R
- added R14, R15: 4.7k, Resistors_SMD:R_0603, symbol R_Small
- added R6: 270, Resistors_SMD:R_0603, symbol R
- added R7, R8: 1k, Resistors_SMD:R_0603, symbol R
- added SW1: SWITCH_DPDT, Synapse:SO-DPDT-6, symbol SWITCH_DPDT
- added SW2, SW3, SW4: SW_PUSH, Buttons_Switches_SMD:SW_SPST_PTS645, symbol SW_PUSH
- added U4: LD1117S33CTR, TO_SOT_Packages_SMD:SOT-223, symbol LD1117S33CTR
- added U5: LIS3DH, Synapse:LGA16_3x3, symbol LIS3DH
- C1: renamed from C?; footprint (none) -> Capacitors_SMD:C_0603
- D1: footprint LEDs:LED-0603 -> w_smd_leds:Led_0603
- D65, D66: renamed from D?; footprint LEDs:LED-0603 -> w_smd_leds:Led_0603
- FB1: renamed from FB?; value FILTER -> 600 OHM 500MA; footprint (none) -> Resistors_SMD:R_0603
- R2, R3, R4, R5: renamed from R?; footprint (none) -> Resistors_SMD:R_0603
- U3: renamed from U?; footprint SSOP-16 -> Housings_SSOP:SSOP-16_3.9x4.9mm_Pitch0.635mm
Connections:
- net labels added: *IS_USB, *RESET, ACC_INT1, ACC_INT2, BTN_LFT, BTN_RT, I2C_SCL, I2C_SDA, LED_PWR_EN, PB0, PB5, PB6, PB7, PD4, PE0, PE1, PE3, PE4, PE5, PE7, PF0, PF1, PF4, PF5, PF6, PF7, STATUS_LED, VIN_USB, VREG_IN
- net labels removed: DIG0, DIG1, DIG2, DIG3, DIG4, DIG5, DIG6, DIG7, LED_LD, SEGA, SEGB, SEGC, SEGD, SEGDP, SEGE, SEGF, SEGG
- wire segments 134 -> 188
- no-connect marks 34 -> 9
Other:
- note added: "AAA battery\n holders"
- note added: "AD0"
- note added: "AD1"
- note added: "AD2"
- note added: "AD3"
- note added: "AD4"
- note added: "AD5"
- note added: "AREF"
- note added: "Accelerometer"
- note added: "Arduino Shield\n Connectors\n\n!! 3.3V ONLY !!"
- note added: "D0 RXD"
- note added: "D1 TXD"
- note added: "D10"
- note added: "D2"
- note added: "D3"
- note added: "D4"
- note added: "D5"
- note added: "D6"
- note added: "D7"
- note added: "D8"
- note added: "D9"
- note added: "FT230X"
- note added: "GND"
- note added: "I2C ADDR \nRead=0x31 \nWrite=0x30"
- note added: "LIS3DH"
- note added: "Label TX/RX reversed\non silkscreen to indicate\nlocal perspective"
- note added: "MISO"
- note added: "MOSI"
- note added: "PWR Select\nBATT/USB"
- note added: "Radio Module / System Controller"
- note added: "Reverse polarity protection"
- note added: "SCK"
- note added: "SCL"
- note added: "SDA"
- note added: "SM220"
- note added: "USB / Serial Interface"
- note added: "USB Inrush Limiter"
- moved on the sheet: C1, D65, D66, FB1, R2, R3, R4, R5, U1, U3

Commit message: First placement
Parts:
- P1: Kcost (none) -> 0.20; PN (none) -> 10118194-0001LF
- Q1: Kcost (none) -> 0.15; PN (none) -> ZXMN2F30FHTA
- Q2: Kcost (none) -> 0.14; PN (none) -> SI2305CDS-T1-GE3
- U3: Kcost (none) -> 1.53; PN (none) -> FT230XS-R
- U4: Kcost (none) -> 0.14
- U5: Kcost (none) -> 0.80; PN (none) -> LIS3DHTR
Changed lines of the file:
@@
 $EndDescr
 $Comp
-L VCC #PWR8
+L VCC #PWR01
 U 1 1 564B5908
 P 3700 2750
-F 0 "#PWR8" H 3700 2600 50  0001 C CNN
+F 0 "#PWR01" H 3700 2600 50  0001 C CNN
 F 1 "VCC" H 3700 2900 50  0000 C CNN
 F 2 "" H 3700 2750 60  0000 C CNN
@@
 $EndComp
 $Comp
-L GND #PWR9
+L GND #PWR02
 U 1 1 564B591E
 P 3900 3100
-F 0 "#PWR9" H 3900 2850 50  0001 C CNN
+F 0 "#PWR02" H 3900 2850 50  0001 C CNN
 F 1 "GND" H 3900 2950 50  0000 C CNN
 F 2 "" H 3900 3100 60  0000 C CNN
@@
 NoConn ~ 4250 2750
 $Comp
-L PWR_FLAG #FLG2
+L PWR_FLAG #FLG03
 U 1 1 564B5E55
 P 1850 800
-F 0 "#FLG2" H 1850 895 50  0001 C CNN
+F 0 "#FLG03" H 1850 895 50  0001 C CNN
 F 1 "PWR_FLAG" H 1850 980 50  0000 C CNN
 F 2 "" H 1850 800 60  0000 C CNN
@@
 $EndComp
 $Comp
-L PWR_FLAG #FLG3
+L PWR_FLAG #FLG04
 U 1 1 564B5E6C
 P 2350 800
-F 0 "#FLG3" H 2350 895 50  0001 C CNN
+F 0 "#FLG04" H 2350 895 50  0001 C CNN
 F 1 "PWR_FLAG" H 2350 980 50  0000 C CNN
 F 2 "" H 2350 800 60  0000 C CNN
@@
 $EndComp
 $Comp
-L GND #PWR2
+L GND #PWR05
 U 1 1 564B5E82
 P 1850 850
-F 0 "#PWR2" H 1850 600 50  0001 C CNN
+F 0 "#PWR05" H 1850 600 50  0001 C CNN
 F 1 "GND" H 1850 700 50  0000 C CNN
 F 2 "" H 1850 850 60  0000 C CNN
@@
 $EndComp
 $Comp
-L VCC #PWR5
+L VCC #PWR06
 U 1 1 564B5E98
 P 2350 850
-F 0 "#PWR5" H 2350 700 50  0001 C CNN
+F 0 "#PWR06" H 2350 700 50  0001 C CNN
 F 1 "VCC" H 2350 1000 50  0000 C CNN
 F 2 "" H 2350 850 60  0000 C CNN
@@
 F 1 "FT230XS" H 9500 6050 60  0000 C CNN
 F 2 "Housings_SSOP:SSOP-16_3.9x4.9mm_Pitch0.635mm" H 9150 5500 60  0001 C CNN
-F 3 "" H 9150 5500 60  0000 C CNN
+F 3 "http://www.digikey.com/product-detail/en/FT230XS-R/768-1135-1-ND/3029155" H 9150 5500 60  0001 C CNN
+F 4 "1.53" H 9150 5500 60  0001 C CNN "Kcost"
+F 5 "FT230XS-R" H 9150 5500 60  0001 C CNN "PN"
 	1    9150 5500
 	1    0    0    -1
@@
 $EndComp
 $Comp
-L GND #PWR17
+L GND #PWR07
 U 1 1 564FF241
 P 6750 6050
-F 0 "#PWR17" H 6750 5800 50  0001 C CNN
+F 0 "#PWR07" H 6750 5800 50  0001 C CNN
 F 1 "GND" H 6750 5900 50  0000 C CNN
 F 2 "" H 6750 6050 60  0000 C CNN
@@
 $EndComp
 $Comp
-L GND #PWR20
+L GND #PWR08
 U 1 1 56506EFF
 P 8200 6300
-F 0 "#PWR20" H 8200 6050 50  0001 C CNN
+F 0 "#PWR08" H 8200 6050 50  0001 C CNN
 F 1 "GND" H 8200 6150 50  0000 C CNN
 F 2 "" H 8200 6300 60  0000 C CNN
@@
 F 1 "LD1117S33CTR" H 1650 7100 40  0000 C CNN
 F 2 "TO_SOT_Packages_SMD:SOT-223" H 1650 7000 40  0001 C CNN
-F 3 "" H 1650 6900 60  0000 C CNN
+F 3 "http://www.digikey.com/product-detail/en/LD1117S33CTR/497-1241-1-ND/586241" H 1650 6900 60  0001 C CNN
+F 4 "0.14" H 1650 6900 60  0001 C CNN "Kcost"
 	1    1650 6900
 	1    0    0    -1
@@
 $EndComp
 $Comp
-L GND #PWR1
+L GND #PWR09
 U 1 1 5651B918
 P 1650 7400
-F 0 "#PWR1" H 1650 7150 50  0001 C CNN
+F 0 "#PWR09" H 1650 7150 50  0001 C CNN
 F 1 "GND" H 1650 7250 50  0000 C CNN
 F 2 "" H 1650 7400 60  0000 C CNN
@@
 $EndSheet
 $Comp
-L PWR_FLAG #FLG1
+L PWR_FLAG #FLG010
 U 1 1 5652EBF3
 P 800 6650
-F 0 "#FLG1" H 800 6745 50  0001 C CNN
+F 0 "#FLG010" H 800 6745 50  0001 C CNN
 F 1 "PWR_FLAG" H 800 6830 50  0000 C CNN
 F 2 "" H 800 6650 60  0000 C CNN
@@
 $EndComp
 $Comp
-L GND #PWR6
+L GND #PWR011
 U 1 1 5652F503
 P 2550 5900
-F 0 "#PWR6" H 2550 5650 50  0001 C CNN
+F 0 "#PWR011" H 2550 5650 50  0001 C CNN
 F 1 "GND" H 2550 5750 50  0000 C CNN
 F 2 "" H 2550 5900 60  0000 C CNN
@@
 Reverse polarity protection
 $Comp
-L VCC #PWR10
+L VCC #PWR012
 U 1 1 5653CA88
 P 4100 6650
-F 0 "#PWR10" H 4100 6500 50  0001 C CNN
+F 0 "#PWR012" H 4100 6500 50  0001 C CNN
 F 1 "VCC" H 4100 6800 50  0000 C CNN
 F 2 "" H 4100 6650 60  0000 C CNN
@@
 $EndComp
 $Comp
-L GND #PWR7
+L GND #PWR013
 U 1 1 5653DE03
 P 2800 7400
-F 0 "#PWR7" H 2800 7150 50  0001 C CNN
+F 0 "#PWR013" H 2800 7150 50  0001 C CNN
 F 1 "GND" H 2800 7250 50  0000 C CNN
 F 2 "" H 2800 7400 60  0000 C CNN
@@
 F 1 "LIS3DH" H 9700 1700 60  0000 C CNN
 F 2 "Synapse:LGA16_3x3" H 9650 1750 60  0001 C CNN
-F 3 "" H 9650 1750 60  0000 C CNN
+F 3 "http://www.digikey.com/product-detail/en/LIS3DHTR/497-10613-1-ND/2334355" H 9650 1750 60  0001 C CNN
+F 4 "LIS3DHTR" H 9650 1750 60  0001 C CNN "PN"
+F 5 "0.80" H 9650 1750 60  0001 C CNN "Kcost"
 	1    9650 1750
 	1    0    0    -1
 $EndComp
 $Comp
-L GND #PWR22
+L GND #PWR014
 U 1 1 5654CDCB
 P 9850 2600
-F 0 "#PWR22" H 9850 2350 50  0001 C CNN
+F 0 "#PWR014" H 9850 2350 50  0001 C CNN
 F 1 "GND" H 9850 2450 50  0000 C CNN
 F 2 "" H 9850 2600 60  0000 C CNN
@@
 $EndComp
 $Comp
-L VCC #PWR23
+L VCC #PWR015
 U 1 1 5654D421
 P 9950 900
-F 0 "#PWR23" H 9950 750 50  0001 C CNN
+F 0 "#PWR015" H 9950 750 50  0001 C CNN
 F 1 "VCC" H 9950 1050 50  0000 C CNN
 F 2 "" H 9950 900 60  0000 C CNN
@@
 $EndComp
 $Comp
-L GND #PWR13
+L GND #PWR016
 U 1 1 5655B0D8
 P 4800 7550
-F 0 "#PWR13" H 4800 7300 50  0001 C CNN
+F 0 "#PWR016" H 4800 7300 50  0001 C CNN
 F 1 "GND" H 4800 7400 50  0000 C CNN
 F 2 "" H 4800 7550 60  0000 C CNN
@@
 $EndComp
 $Comp
-L VCC #PWR12
+L VCC #PWR017
 U 1 1 5655B12B
 P 4800 7000
-F 0 "#PWR12" H 4800 6850 50  0001 C CNN
+F 0 "#PWR017" H 4800 6850 50  0001 C CNN
 F 1 "VCC" H 4800 7150 50  0000 C CNN
 F 2 "" H 4800 7000 60  0000 C CNN
@@
 $EndComp
 $Comp
-L GND #PWR15
+L GND #PWR018
 U 1 1 565603AD
 P 5500 7550
-F 0 "#PWR15" H 5500 7300 50  0001 C CNN
+F 0 "#PWR018" H 5500 7300 50  0001 C CNN
 F 1 "GND" H 5500 7400 50  0000 C CNN
 F 2 "" H 5500 7550 60  0000 C CNN
@@
 $EndComp
 $Comp
-L VCC #PWR14
+L VCC #PWR019
 U 1 1 565603B3
 P 5500 7000
-F 0 "#PWR14" H 5500 6850 50  0001 C CNN
+F 0 "#PWR019" H 5500 6850 50  0001 C CNN
 F 1 "VCC" H 5500 7150 50  0000 C CNN
 F 2 "" H 5500 7000 60  0000 C CNN
@@
 $EndComp
 $Comp
-L GND #PWR16
+L GND #PWR020
 U 1 1 56560696
 P 6150 7550
-F 0 "#PWR16" H 6150 7300 50  0001 C CNN
+F 0 "#PWR020" H 6150 7300 50  0001 C CNN
 F 1 "GND" H 6150 7400 50  0000 C CNN
 F 2 "" H 6150 7550 60  0000 C CNN
@@
 $EndComp
 $Comp
-L GND #PWR21
+L GND #PWR021
 U 1 1 5656F8A3
 P 9750 4050
-F 0 "#PWR21" H 9750 3800 50  0001 C CNN
+F 0 "#PWR021" H 9750 3800 50  0001 C CNN
 F 1 "GND" H 9750 3900 50  0000 C CNN
 F 2 "" H 9750 4050 60  0000 C CNN
@@
 $EndComp
 $Comp
-L VCC #PWR19
+L VCC #PWR022
 U 1 1 5657393A
 P 7750 1950
-F 0 "#PWR19" H 7750 1800 50  0001 C CNN
+F 0 "#PWR022" H 7750 1800 50  0001 C CNN
 F 1 "VCC" H 7750 2100 50  0000 C CNN
 F 2 "" H 7750 1950 60  0000 C CNN
@@
 *RESET
 $Comp
-L VCC #PWR3
+L VCC #PWR023
 U 1 1 56588A1C
 P 2150 4250
-F 0 "#PWR3" H 2150 4100 50  0001 C CNN
+F 0 "#PWR023" H 2150 4100 50  0001 C CNN
 F 1 "VCC" H 2150 4400 50  0000 C CNN
 F 2 "" H 2150 4250 60  0000 C CNN
@@
 $EndComp
 $Comp
-L GND #PWR4
+L GND #PWR024
 U 1 1 56588BF1
 P 2150 4500
-F 0 "#PWR4" H 2150 4250 50  0001 C CNN
+F 0 "#PWR024" H 2150 4250 50  0001 C CNN
 F 1 "GND" H 2150 4350 50  0000 C CNN
 F 2 "" H 2150 4500 60  0000 C CNN
@@
 F 1 "Si2305DS" V 4150 5250 50  0000 R CNN
 F 2 "TO_SOT_Packages_SMD:SOT-23" H 4400 4850 29  0001 C CNN
-F 3 "" H 4200 4750 60  0000 C CNN
+F 3 "http://www.digikey.com/product-detail/en/SI2305CDS-T1-GE3/SI2305CDS-T1-GE3CT-ND/3758764" H 4200 4750 60  0001 C CNN
+F 4 "0.14" V 4200 4750 60  0001 C CNN "Kcost"
+F 5 "SI2305CDS-T1-GE3" V 4200 4750 60  0001 C CNN "PN"
 	1    4200 4750
 	0    1    -1   0
@@
 $EndComp
 $Comp
-L GND #PWR11
+L GND #PWR025
 U 1 1 565F01D7
 P 4200 5650
-F 0 "#PWR11" H 4200 5400 50  0001 C CNN
+F 0 "#PWR025" H 4200 5400 50  0001 C CNN
 F 1 "GND" H 4200 5500 50  0000 C CNN
 F 2 "" H 4200 5650 60  0000 C CNN
@@
 F 1 "ZXMN2F30FHCT-ND" V 2100 6050 50  0000 R CNN
 F 2 "TO_SOT_Packages_SMD:SOT-23" H 2050 5800 29  0001 C CNN
-F 3 "" H 1850 5700 60  0000 C CNN
+F 3 "http://www.digikey.com/product-search/en?keywords=ZXMN2F30FHCT-ND" H 1850 5700 60  0001 C CNN
+F 4 "0.15" V 1850 5700 60  0001 C CNN "Kcost"
+F 5 "ZXMN2F30FHTA" V 1850 5700 60  0001 C CNN "PN"
 	1    1850 5700
 	0    -1   1    0
@@
 $EndComp
 $Comp
-L VCC #PWR18
+L VCC #PWR026
 U 1 1 565F68F0
 P 7200 750
-F 0 "#PWR18" H 7200 600 50  0001 C CNN
+F 0 "#PWR026" H 7200 600 50  0001 C CNN
 F 1 "VCC" H 7200 900 50  0000 C CNN
 F 2 "" H 7200 750 60  0000 C CNN
@@
 F 1 "MicroB" H 6300 5700 50  0000 C CNN
 F 2 "Synapse:USBmicroB" V 6250 5400 60  0001 C CNN
-F 3 "" V 6250 5400 60  0000 C CNN
+F 3 "http://www.digikey.com/product-detail/en/10118194-0001LF/609-4618-2-ND/2785389" V 6250 5400 60  0001 C CNN
+F 4 "0.20" H 6300 5500 60  0001 C CNN "Kcost"
+F 5 "10118194-0001LF" H 6300 5500 60  0001 C CNN "PN"
 	1    6300 5500
 	0    -1   1    0

Commit message: Placement v1
Parts:
- P2, P3: footprint Pin_Headers:Pin_Header_Straight_1x08 -> Socket_Strips:Socket_Strip_Straight_1x08
- P4: footprint Pin_Headers:Pin_Header_Straight_1x10 -> Socket_Strips:Socket_Strip_Straight_1x10
- P5: footprint Pin_Headers:Pin_Header_Straight_1x06 -> Socket_Strips:Socket_Strip_Straight_1x06
Changed lines of the file:
@@
 F 0 "P2" H 1300 3200 50  0000 C CNN
 F 1 "CONN_01X08" V 1400 2750 50  0000 C CNN
-F 2 "Pin_Headers:Pin_Header_Straight_1x08" H 1300 2750 60  0001 C CNN
+F 2 "Socket_Strips:Socket_Strip_Straight_1x08" H 1300 2750 60  0001 C CNN
 F 3 "" H 1300 2750 60  0000 C CNN
 	1    1300 2750
@@
 F 0 "P3" H 2450 3950 50  0000 C CNN
 F 1 "CONN_01X08" V 2550 3500 50  0000 C CNN
-F 2 "Pin_Headers:Pin_Header_Straight_1x08" H 2450 3500 60  0001 C CNN
+F 2 "Socket_Strips:Socket_Strip_Straight_1x08" H 2450 3500 60  0001 C CNN
 F 3 "" H 2450 3500 60  0000 C CNN
 	1    2450 3500
@@
 F 0 "P4" H 2450 2950 50  0000 C CNN
 F 1 "CONN_01X10" V 2550 2400 50  0000 C CNN
-F 2 "Pin_Headers:Pin_Header_Straight_1x10" H 2450 2400 60  0001 C CNN
+F 2 "Socket_Strips:Socket_Strip_Straight_1x10" H 2450 2400 60  0001 C CNN
 F 3 "" H 2450 2400 60  0000 C CNN
 	1    2450 2400
@@
 F 0 "P5" H 1300 3950 50  0000 C CNN
 F 1 "CONN_01X06" V 1400 3600 50  0000 C CNN
-F 2 "Pin_Headers:Pin_Header_Straight_1x06" H 1300 3600 60  0001 C CNN
+F 2 "Socket_Strips:Socket_Strip_Straight_1x06" H 1300 3600 60  0001 C CNN
 F 3 "" H 1300 3600 60  0000 C CNN
 	1    1300 3600

Commit message: Backup
Changed lines of the file:
@@
 FT230X
 Text Label 6150 6900 0    60   ~ 0
-VREG_IN
+VIN_USB
 $Comp
 L SW_PUSH SW2

Commit message: Placement complete.
Parts:
- added R16: 4.7k, Resistors_SMD:R_0603, symbol R
Connections:
- wire segments 188 -> 192
- no-connect marks 9 -> 7
Changed lines of the file:
@@
 	1    0    0    -1
 $EndComp
-NoConn ~ 4250 2750
 $Comp
 L PWR_FLAG #FLG03
@@
 PD4
 Wire Wire Line
-	3900 2950 3900 3100
+	3900 2750 3900 3100
 Wire Wire Line
 	1850 800  1850 850
@@
 	6350 1350 6800 1350
 Wire Wire Line
-	6950 1250 6350 1250
+	6350 1250 6950 1250
 Wire Wire Line
 	6350 2650 6800 2650
@@
 Text Label 6400 2650 0    60   ~ 0
 PB6
-NoConn ~ 4250 1450
 NoConn ~ 4250 2150
 Wire Wire Line
@@
 Wire Wire Line
 	6200 5900 6200 5950
+$Comp
+L GND #PWR027
+U 1 1 5669638E
+P 3650 2000
+F 0 "#PWR027" H 3650 1750 50  0001 C CNN
+F 1 "GND" H 3650 1850 50  0000 C CNN
+F 2 "" H 3650 2000 60  0000 C CNN
+F 3 "" H 3650 2000 60  0000 C CNN
+	1    3650 2000
+	1    0    0    -1
+$EndComp
+Wire Wire Line
+	3650 1900 3650 2000
+Wire Wire Line
+	4250 2750 3900 2750
+Connection ~ 3900 2950
+$Comp
+L R R16
+U 1 1 56698EE9
+P 3650 1750
+F 0 "R16" V 3730 1750 50  0000 C CNN
+F 1 "4.7k" V 3650 1750 50  0000 C CNN
+F 2 "Resistors_SMD:R_0603" V 3580 1750 30  0001 C CNN
+F 3 "" H 3650 1750 30  0000 C CNN
+	1    3650 1750
+	1    0    0    -1
+$EndComp
+Wire Wire Line
+	4250 1450 3650 1450
+Wire Wire Line
+	3650 1450 3650 1600
 $EndSCHEMATC

Commit message: First version sent to CM for review (Screaming Circuits)
Parts:
- BT1, BT2: Kcost (none) -> .59; PN (none) -> 2466
- C1, C2, C21, C4, C5, C6: PN (none) -> X5R/X7R, 50V
- C10, C12, C20: PN (none) -> X5R/X7R, 16V
- C11, C15, C22, C23, C3, C7, C8, C9: PN (none) -> X5R/X7R, 6.3V
- FB1: Kcost (none) -> .07; PN (none) -> BLM18EG601SN1D
- P2, P3: Kcost (none) -> .64; PN (none) -> FCI 75915-308LF
- P4: Kcost (none) -> .78; PN (none) -> FCI 75915-310LF
- P5: Kcost (none) -> .49; PN (none) -> FCI 75915-306LF
- P6: Kcost (none) -> .58; PN (none) -> FCI 87606-303LF
- U1: Kcost (none) -> 20.00; PN (none) -> SM220UF1
Changed lines of the file:
@@
 F 1 "600 OHM 500MA" H 7750 4900 50  0000 C CNN
 F 2 "Resistors_SMD:R_0603" H 7750 5000 60  0001 C CNN
-F 3 "BLM18EG601SN1D" H 7750 5000 60  0001 C CNN
+F 3 "http://www.digikey.com/product-detail/en/BLM18EG601SN1D/490-3994-1-ND/1016254" H 7750 5000 60  0001 C CNN
+F 4 "BLM18EG601SN1D" H 7750 5000 60  0001 C CNN "PN"
+F 5 ".07" H 7750 5000 60  0001 C CNN "Kcost"
 	1    7750 5000
 	1    0    0    -1
@@
 F 2 "Capacitors_SMD:C_0603" H 8238 5800 30  0001 C CNN
 F 3 "" H 8200 5950 60  0000 C CNN
+F 4 "X5R/X7R, 50V " H 8200 5950 60  0001 C CNN "PN"
 	1    8200 5950
 	1    0    0    -1
@@
 F 2 "Capacitors_SMD:C_0603" H 1138 7050 30  0001 C CNN
 F 3 "" H 1100 7200 60  0000 C CNN
+F 4 "X5R/X7R, 50V " H 1100 7200 60  0001 C CNN "PN"
 	1    1100 7200
 	1    0    0    -1
@@
 	1    1650 7400
 	1    0    0    -1
-$EndComp
-$Comp
-L Battery BT1
-U 1 1 5652075D
-P 1400 5650
-F 0 "BT1" H 1500 5700 50  0000 L CNN
-F 1 "1.5V" H 1500 5600 50  0000 L CNN
-F 2 "Synapse:BATT_2466" V 1400 5690 60  0001 C CNN
-F 3 "" V 1400 5690 60  0000 C CNN
-	1    1400 5650
-	-1   0    0    -1
 $EndComp
 $Sheet
@@
 F 2 "Capacitors_SMD:C_0603" H 6900 5700 60  0001 C CNN
 F 3 "" H 6900 5700 60  0000 C CNN
+F 4 "X5R/X7R, 50V " H 6900 5700 60  0001 C CNN "PN"
 	1    6900 5700
 	1    0    0    -1
@@
 F 2 "Capacitors_SMD:C_0603" H 7150 5700 60  0001 C CNN
 F 3 "" H 7150 5700 60  0000 C CNN
+F 4 "X5R/X7R, 50V " H 7150 5700 60  0001 C CNN "PN"
 	1    7150 5700
 	1    0    0    -1
@@
 F 2 "Capacitors_SMD:C_0603" H 7400 5700 60  0001 C CNN
 F 3 "" H 7400 5700 60  0000 C CNN
+F 4 "X5R/X7R, 50V " H 7400 5700 60  0001 C CNN "PN"
 	1    7400 5700
 	1    0    0    -1
@@
 F 1 "1.5V" H 1500 5250 50  0000 L CNN
 F 2 "Synapse:BATT_2466" V 1400 5340 60  0001 C CNN
-F 3 "" V 1400 5340 60  0000 C CNN
+F 3 "http://www.digikey.com/product-detail/en/2466/36-2466-ND/303815" V 1400 5340 60  0001 C CNN
+F 4 ".59" H 1400 5300 60  0001 C CNN "Kcost"
+F 5 "2466" H 1400 5300 60  0001 C CNN "PN"
 	1    1400 5300
 	-1   0    0    -1
@@
 F 2 "Capacitors_SMD:C_0603" H 2188 7050 30  0001 C CNN
 F 3 "" H 2150 7200 60  0000 C CNN
+F 4 "X5R/X7R, 6.3V " H 2150 7200 60  0001 C CNN "PN"
 	1    2150 7200
 	1    0    0    -1
@@
 F 2 "Capacitors_SMD:C_0603" H 4838 7150 30  0001 C CNN
 F 3 "" H 4800 7300 60  0000 C CNN
+F 4 "X5R/X7R, 6.3V " H 4800 7300 60  0001 C CNN "PN"
 	1    4800 7300
 	1    0    0    -1
@@
 F 2 "Capacitors_SMD:C_0603" H 5538 7150 30  0001 C CNN
 F 3 "" H 5500 7300 60  0000 C CNN
+F 4 "X5R/X7R, 6.3V " H 5500 7300 60  0001 C CNN "PN"
 	1    5500 7300
 	1    0    0    -1
@@
 F 2 "Capacitors_SMD:C_0603" H 5838 7150 30  0001 C CNN
 F 3 "" H 5800 7300 60  0000 C CNN
+F 4 "X5R/X7R, 16V " H 5800 7300 60  0001 C CNN "PN"
 	1    5800 7300
 	1    0    0    -1
@@
 F 2 "Capacitors_SMD:C_0603" H 6188 7150 30  0001 C CNN
 F 3 "" H 6150 7300 60  0000 C CNN
+F 4 "X5R/X7R, 6.3V " H 6150 7300 60  0001 C CNN "PN"
 	1    6150 7300
 	1    0    0    -1
@@
 F 2 "Capacitors_SMD:C_0603" H 6488 7150 30  0001 C CNN
 F 3 "" H 6450 7300 60  0000 C CNN
+F 4 "X5R/X7R, 16V " H 6450 7300 60  0001 C CNN "PN"
 	1    6450 7300
 	1    0    0    -1
@@
 F 1 "CONN_01X08" V 1400 2750 50  0000 C CNN
 F 2 "Socket_Strips:Socket_Strip_Straight_1x08" H 1300 2750 60  0001 C CNN
-F 3 "" H 1300 2750 60  0000 C CNN
+F 3 "http://www.digikey.com/product-detail/en/75915-308LF/609-3559-ND/1523940" H 1300 2750 60  0001 C CNN
+F 4 "FCI 75915-308LF" H 1300 2750 60  0001 C CNN "PN"
+F 5 ".64" H 1300 2750 60  0001 C CNN "Kcost"
 	1    1300 2750
 	1    0    0    -1
@@
 F 1 "CONN_01X08" V 2550 3500 50  0000 C CNN
 F 2 "Socket_Strips:Socket_Strip_Straight_1x08" H 2450 3500 60  0001 C CNN
-F 3 "" H 2450 3500 60  0000 C CNN
+F 3 "http://www.digikey.com/product-detail/en/75915-308LF/609-3559-ND/1523940" H 2450 3500 60  0001 C CNN
+F 4 "FCI 75915-308LF" H 2450 3500 60  0001 C CNN "PN"
+F 5 ".64" H 2450 3500 60  0001 C CNN "Kcost"
 	1    2450 3500
 	1    0    0    -1
@@
 F 1 "CONN_01X10" V 2550 2400 50  0000 C CNN
 F 2 "Socket_Strips:Socket_Strip_Straight_1x10" H 2450 2400 60  0001 C CNN
-F 3 "" H 2450 2400 60  0000 C CNN
+F 3 "http://www.digikey.com/product-detail/en/75915-310LF/609-3550-ND/1524287" H 2450 2400 60  0001 C CNN
+F 4 ".78" H 2450 2400 60  0001 C CNN "Kcost"
+F 5 "FCI 75915-310LF" H 2450 2400 60  0001 C CNN "PN"
 	1    2450 2400
 	1    0    0    -1
@@
 F 1 "CONN_01X06" V 1400 3600 50  0000 C CNN
 F 2 "Socket_Strips:Socket_Strip_Straight_1x06" H 1300 3600 60  0001 C CNN
-F 3 "" H 1300 3600 60  0000 C CNN
+F 3 "http://www.digikey.com/product-detail/en/75915-306LF/609-3558-ND/1523584" H 1300 3600 60  0001 C CNN
+F 4 ".49" H 1300 3600 60  0001 C CNN "Kcost"
+F 5 "FCI 75915-306LF" H 1300 3600 60  0001 C CNN "PN"
 	1    1300 3600
 	1    0    0    -1
@@
 F 1 "CONN_02X03" H 1750 4150 50  0000 C CNN
 F 2 "Pin_Headers:Pin_Header_Straight_2x03" H 1750 3150 60  0001 C CNN
-F 3 "" H 1750 3150 60  0000 C CNN
+F 3 "http://www.digikey.com/product-detail/en/87606-303LF/87606-303LF-ND/1523609" H 1750 3150 60  0001 C CNN
+F 4 "FCI 87606-303LF" H 1750 4350 60  0001 C CNN "PN"
+F 5 ".58" H 1750 4350 60  0001 C CNN "Kcost"
 	1    1750 4350
 	1    0    0    -1
@@
 F 1 "SM220" H 4800 1200 60  0000 C CNN
 F 2 "Synapse:SM220" H 5100 -800 60  0000 C CNN
-F 3 "" H 4850 1150 60  0000 C CNN
+F 3 "http://www.digikey.com/product-detail/en/SM220UF1/746-1053-1-ND/5171418" H 4850 1150 60  0001 C CNN
+F 4 "SM220UF1" H 4850 1150 60  0001 C CNN "PN"
+F 5 "20.00" H 4850 1150 60  0001 C CNN "Kcost"
 	1    4850 1150
 	1    0    0    -1
@@
 F 2 "Capacitors_SMD:C_0603" H 7888 5800 30  0001 C CNN
 F 3 "" H 7850 5950 60  0000 C CNN
+F 4 "X5R/X7R, 6.3V " H 7850 5950 60  0001 C CNN "PN"
 	1    7850 5950
 	1    0    0    -1
@@
 F 2 "Capacitors_SMD:C_0603" H 2238 5300 30  0001 C CNN
 F 3 "" H 2200 5450 60  0000 C CNN
+F 4 "X5R/X7R, 6.3V " H 2200 5450 60  0001 C CNN "PN"
 	1    2200 5450
 	1    0    0    -1
@@
 F 2 "Capacitors_SMD:C_0603" H 2588 5300 30  0001 C CNN
 F 3 "" H 2550 5450 60  0000 C CNN
+F 4 "X5R/X7R, 16V " H 2550 5450 60  0001 C CNN "PN"
 	1    2550 5450
 	1    0    0    -1
@@
 F 2 "Capacitors_SMD:C_0603" H 3838 4800 30  0001 C CNN
 F 3 "" H 3800 4950 60  0000 C CNN
+F 4 "X5R/X7R, 50V " H 3800 4950 60  0001 C CNN "PN"
 	1    3800 4950
 	1    0    0    -1
@@
 F 2 "Capacitors_SMD:C_0603" H 5138 7150 30  0001 C CNN
 F 3 "" H 5100 7300 60  0000 C CNN
+F 4 "X5R/X7R, 6.3V " H 5100 7300 60  0001 C CNN "PN"
 	1    5100 7300
 	1    0    0    -1
@@
 F 2 "Capacitors_SMD:C_0603" H 4538 7150 30  0001 C CNN
 F 3 "" H 4500 7300 60  0000 C CNN
+F 4 "X5R/X7R, 6.3V " H 4500 7300 60  0001 C CNN "PN"
 	1    4500 7300
 	1    0    0    -1
@@
 Wire Wire Line
 	3650 1450 3650 1600
+$Comp
+L Battery BT1
+U 1 1 5672E2BE
+P 1400 5650
+F 0 "BT1" H 1500 5700 50  0000 L CNN
+F 1 "1.5V" H 1500 5600 50  0000 L CNN
+F 2 "Synapse:BATT_2466" V 1400 5690 60  0001 C CNN
+F 3 "http://www.digikey.com/product-detail/en/2466/36-2466-ND/303815" V 1400 5690 60  0001 C CNN
+F 4 ".59" H 1400 5650 60  0001 C CNN "Kcost"
+F 5 "2466" H 1400 5650 60  0001 C CNN "PN"
+	1    1400 5650
+	-1   0    0    -1
+$EndComp
 $EndSCHEMATC
