File: test_board2.sch (KiCad schematic (older format))
At the start: 51 parts, among them P1 MicroB, P2 CONN_01X08, P3 CONN_01X08, P4 CONN_01X10, P5 CONN_01X06, P6 CONN_02X03, Q1 ZXMN2F30FHCT-ND, Q2 Si2305DS, SW1 SWITCH_DPDT, SW2 SW_PUSH, SW3 SW_PUSH, SW4 SW_PUSH, U1 SM220, U3 FT230XS, U4 LD1117S33CTR, U5 LIS3DH

Commit message: Update sch with Mfg and PN fields, added Screaming Circuits to silk.
Parts:
- BT1, BT2: Mfg (none) -> Keystone
- C1, C2, C21: value 100nF -> 0.1uF; Mfg (none) -> Samsung; PN X5R/X7R, 50V -> CL10B104KB8SFNC; Spec (none) -> X5R/X7R, 50V
- C10, C12, C20: Mfg (none) -> Samsung; PN X5R/X7R, 16V -> CL10B104KB8SFNC; Spec (none) -> X5R/X7R, 16V
- C11, C15, C9: Mfg (none) -> Samsung; PN X5R/X7R, 6.3V -> CL10B475KQ8NQNC; Spec (none) -> X5R/X7R, 6.3V
- C22, C23, C7, C8: Mfg (none) -> Samsung; PN X5R/X7R, 6.3V -> CL10A226MQ8NRNC; Spec (none) -> X5R/X7R, 6.3V
- C3: Mfg (none) -> Samsung; PN X5R/X7R, 6.3V -> CL10A106MQ8NNNC; Spec (none) -> X5R/X7R, 6.3V
- C4: Mfg (none) -> Yageo; PN X5R/X7R, 50V -> CC0603KRX7R9BB103; Spec (none) -> X5R/X7R, 50V
- C5, C6: Mfg (none) -> Samsung; PN X5R/X7R, 50V -> CL10C470JB8NNNC; Spec (none) -> NPO, 50V
- FB1: Mfg (none) -> Murata
- P1, P2, P3, P4, P5: Mfg (none) -> FCI
- P6: Kcost .58 -> .14; Mfg (none) -> FCI; PN FCI 87606-303LF -> FCI 67997-206HLF
- Q1: Mfg (none) -> Diodes Incorporated
- Q2: Mfg (none) -> Vishay Siliconix
- R12: Mfg (none) -> Yageo; PN (none) -> RC0603FR-07100KL
- R13: Mfg (none) -> Yageo; PN (none) -> RC0603FR-0739KL
- R14, R15, R16: Mfg (none) -> Yageo; PN (none) -> RC0603FR-074K7L
- R2, R3: Mfg (none) -> Yageo; PN (none) -> RC0603FR-0727RL
- R4, R5, R6: Mfg (none) -> Yageo; PN (none) -> RC0603FR-07270RL
- R7, R8: Mfg (none) -> Yageo; PN (none) -> RC0603FR-071KL
- SW1, SW2, SW3, SW4: Mfg (none) -> C&K Components
- U1: Mfg (none) -> Synapse Wireless
- U3: Mfg (none) -> FTDI
- U4: Mfg (none) -> ST Microelectronics; PN (none) -> LD1117S33CTR
- U5: Mfg (none) -> ST Microelectronics
