File: LED_matrix.sch (KiCad schematic (older format))
At the start: 87 parts, among them SW5 SW_DIP_8, U2 AS1115, U6 TPS61070, U7 NLSX4373

Commit message: First placement
Parts:
- U7: Kcost (none) -> 0.40; PN (none) -> NLSX4373
Changed lines of the file:
@@
 $EndComp
 $Comp
-L GND #PWR27
+L GND #PWR027
 U 1 1 56568DD7
 P 6350 7500
-F 0 "#PWR27" H 6350 7250 50  0001 C CNN
+F 0 "#PWR027" H 6350 7250 50  0001 C CNN
 F 1 "GND" H 6350 7350 50  0000 C CNN
 F 2 "" H 6350 7500 60  0000 C CNN
@@
 $EndComp
 $Comp
-L GND #PWR28
+L GND #PWR028
 U 1 1 565ABD42
 P 6800 4900
-F 0 "#PWR28" H 6800 4650 50  0001 C CNN
+F 0 "#PWR028" H 6800 4650 50  0001 C CNN
 F 1 "GND" H 6800 4750 50  0000 C CNN
 F 2 "" H 6800 4900 60  0000 C CNN
@@
 $EndComp
 $Comp
-L GND #PWR26
+L GND #PWR029
 U 1 1 565ABE47
 P 6250 5450
-F 0 "#PWR26" H 6250 5200 50  0001 C CNN
+F 0 "#PWR029" H 6250 5200 50  0001 C CNN
 F 1 "GND" H 6250 5300 50  0000 C CNN
 F 2 "" H 6250 5450 60  0000 C CNN
@@
 $EndComp
 $Comp
-L GND #PWR29
+L GND #PWR030
 U 1 1 565ABF45
 P 6800 5750
-F 0 "#PWR29" H 6800 5500 50  0001 C CNN
+F 0 "#PWR030" H 6800 5500 50  0001 C CNN
 F 1 "GND" H 6800 5600 50  0000 C CNN
 F 2 "" H 6800 5750 60  0000 C CNN
@@
 $EndComp
 $Comp
-L GND #PWR30
+L GND #PWR031
 U 1 1 565AD0B9
 P 7500 4900
-F 0 "#PWR30" H 7500 4650 50  0001 C CNN
+F 0 "#PWR031" H 7500 4650 50  0001 C CNN
 F 1 "GND" H 7500 4750 50  0000 C CNN
 F 2 "" H 7500 4900 60  0000 C CNN
@@
 $EndComp
 $Comp
-L GND #PWR25
+L GND #PWR032
 U 1 1 565AD1C0
 P 5150 5100
-F 0 "#PWR25" H 5150 4850 50  0001 C CNN
+F 0 "#PWR032" H 5150 4850 50  0001 C CNN
 F 1 "GND" H 5150 4950 50  0000 C CNN
 F 2 "" H 5150 5100 60  0000 C CNN
@@
 F 1 "NLSX4373" H 9450 5550 60  0000 C CNN
 F 2 "Housings_SOIC:SOIC-8_3.9x4.9mm_Pitch1.27mm" H 9600 5600 60  0001 C CNN
-F 3 "" H 9600 5600 60  0000 C CNN
+F 3 "http://www.digikey.com/product-detail/en/NLSX4373DR2G/NLSX4373DR2GOSCT-ND/3462432" H 9600 5600 60  0001 C CNN
+F 4 "0.40" H 9600 5600 60  0001 C CNN "Kcost"
+F 5 "NLSX4373" H 9600 5600 60  0001 C CNN "PN"
 	1    9600 5600
 	1    0    0    -1
 $EndComp
 $Comp
-L GND #PWR32
+L GND #PWR033
 U 1 1 56601EAF
 P 8800 6150
-F 0 "#PWR32" H 8800 5900 50  0001 C CNN
+F 0 "#PWR033" H 8800 5900 50  0001 C CNN
 F 1 "GND" H 8800 6000 50  0000 C CNN
 F 2 "" H 8800 6150 60  0000 C CNN
@@
 I2C_SCL
 $Comp
-L VCC #PWR24
+L VCC #PWR034
 U 1 1 56602696
 P 4850 4050
-F 0 "#PWR24" H 4850 3900 50  0001 C CNN
+F 0 "#PWR034" H 4850 3900 50  0001 C CNN
 F 1 "VCC" H 4850 4200 50  0000 C CNN
 F 2 "" H 4850 4050 60  0000 C CNN
@@
 $EndComp
 $Comp
-L VCC #PWR31
+L VCC #PWR035
 U 1 1 566027AD
 P 8800 5600
-F 0 "#PWR31" H 8800 5450 50  0001 C CNN
+F 0 "#PWR035" H 8800 5450 50  0001 C CNN
 F 1 "VCC" H 8800 5750 50  0000 C CNN
 F 2 "" H 8800 5600 60  0000 C CNN

Commit message: Placement v1
Parts:
- D2, D69, D70, D71, D72, D73, D74, D75: footprint Diodes_SMD:SOD-123 -> Diodes_SMD:SOD-323
Changed lines of the file:
@@
 F 0 "D2" H 6550 1230 50  0000 L CNN
 F 1 "1N4148W" H 6450 1070 50  0000 L CNN
-F 2 "Diodes_SMD:SOD-123" V 6600 1150 60  0001 C CNN
+F 2 "Diodes_SMD:SOD-323" V 6600 1150 60  0001 C CNN
 F 3 "http://www.digikey.com/product-detail/en/1N4148W-7-F/1N4148W-FDITR-ND/814371" V 6600 1150 60  0001 C CNN
 F 4 "0.03" H 6600 1150 60  0001 C CNN "Kcost"
@@
 F 0 "D69" H 6550 1480 50  0000 L CNN
 F 1 "1N4148W" H 6450 1320 50  0000 L CNN
-F 2 "Diodes_SMD:SOD-123" V 6600 1400 60  0001 C CNN
+F 2 "Diodes_SMD:SOD-323" V 6600 1400 60  0001 C CNN
 F 3 "http://www.digikey.com/product-detail/en/1N4148W-7-F/1N4148W-FDITR-ND/814371" V 6600 1400 60  0001 C CNN
 F 4 "0.03" H 6600 1400 60  0001 C CNN "Kcost"
@@
 F 0 "D70" H 6550 1730 50  0000 L CNN
 F 1 "1N4148W" H 6450 1570 50  0000 L CNN
-F 2 "Diodes_SMD:SOD-123" V 6600 1650 60  0001 C CNN
+F 2 "Diodes_SMD:SOD-323" V 6600 1650 60  0001 C CNN
 F 3 "http://www.digikey.com/product-detail/en/1N4148W-7-F/1N4148W-FDITR-ND/814371" V 6600 1650 60  0001 C CNN
 F 4 "0.03" H 6600 1650 60  0001 C CNN "Kcost"
@@
 F 0 "D71" H 6550 1980 50  0000 L CNN
 F 1 "1N4148W" H 6450 1820 50  0000 L CNN
-F 2 "Diodes_SMD:SOD-123" V 6600 1900 60  0001 C CNN
+F 2 "Diodes_SMD:SOD-323" V 6600 1900 60  0001 C CNN
 F 3 "http://www.digikey.com/product-detail/en/1N4148W-7-F/1N4148W-FDITR-ND/814371" V 6600 1900 60  0001 C CNN
 F 4 "0.03" H 6600 1900 60  0001 C CNN "Kcost"
@@
 F 0 "D72" H 6550 2230 50  0000 L CNN
 F 1 "1N4148W" H 6450 2070 50  0000 L CNN
-F 2 "Diodes_SMD:SOD-123" V 6600 2150 60  0001 C CNN
+F 2 "Diodes_SMD:SOD-323" V 6600 2150 60  0001 C CNN
 F 3 "http://www.digikey.com/product-detail/en/1N4148W-7-F/1N4148W-FDITR-ND/814371" V 6600 2150 60  0001 C CNN
 F 4 "0.03" H 6600 2150 60  0001 C CNN "Kcost"
@@
 F 0 "D73" H 6550 2480 50  0000 L CNN
 F 1 "1N4148W" H 6450 2320 50  0000 L CNN
-F 2 "Diodes_SMD:SOD-123" V 6600 2400 60  0001 C CNN
+F 2 "Diodes_SMD:SOD-323" V 6600 2400 60  0001 C CNN
 F 3 "http://www.digikey.com/product-detail/en/1N4148W-7-F/1N4148W-FDITR-ND/814371" V 6600 2400 60  0001 C CNN
 F 4 "0.03" H 6600 2400 60  0001 C CNN "Kcost"
@@
 F 0 "D74" H 6550 2730 50  0000 L CNN
 F 1 "1N4148W" H 6450 2570 50  0000 L CNN
-F 2 "Diodes_SMD:SOD-123" V 6600 2650 60  0001 C CNN
+F 2 "Diodes_SMD:SOD-323" V 6600 2650 60  0001 C CNN
 F 3 "http://www.digikey.com/product-detail/en/1N4148W-7-F/1N4148W-FDITR-ND/814371" V 6600 2650 60  0001 C CNN
 F 4 "0.03" H 6600 2650 60  0001 C CNN "Kcost"
@@
 F 0 "D75" H 6550 2980 50  0000 L CNN
 F 1 "1N4148W" H 6450 2820 50  0000 L CNN
-F 2 "Diodes_SMD:SOD-123" V 6600 2900 60  0001 C CNN
+F 2 "Diodes_SMD:SOD-323" V 6600 2900 60  0001 C CNN
 F 3 "http://www.digikey.com/product-detail/en/1N4148W-7-F/1N4148W-FDITR-ND/814371" V 6600 2900 60  0001 C CNN
 F 4 "0.03" H 6600 2900 60  0001 C CNN "Kcost"

Commit message: Backup
Changed lines of the file:
@@
 L SW_DIP_8 SW5
 U 1 1 565CF2D0
-P 7600 2050
-F 0 "SW5" H 7570 2519 60  0000 C CNN
-F 1 "SW_DIP_8" H 7570 1549 60  0000 C CNN
-F 2 "Synapse:DIPSW-16" H 7570 2049 60  0001 C CNN
-F 3 "http://www.digikey.com/product-detail/en/1-1825058-9/1-1825058-9-ND/1021551" H 7570 2049 60  0001 C CNN
-F 4 "1-1825058-9" H 7600 2050 60  0001 C CNN "PN"
-F 5 "0.586" H 7600 2050 60  0001 C CNN "Kcost"
-	1    7600 2050
-	1    0    0    -1
+P 7550 2050
+F 0 "SW5" H 7520 2519 60  0000 C CNN
+F 1 "SW_DIP_8" H 7520 1549 60  0000 C CNN
+F 2 "Synapse:DIPSW-16" H 7520 2049 60  0001 C CNN
+F 3 "http://www.digikey.com/product-detail/en/1-1825058-9/1-1825058-9-ND/1021551" H 7520 2049 60  0001 C CNN
+F 4 "1-1825058-9" H 7550 2050 60  0001 C CNN "PN"
+F 5 "0.586" H 7550 2050 60  0001 C CNN "Kcost"
+	1    7550 2050
+	-1   0    0    -1
 $EndComp
 Wire Wire Line
@@
 Text Label 6300 1150 2    60   ~ 0
 SEGDP
-Connection ~ 7950 1900
-Connection ~ 7950 2000
-Connection ~ 7950 2100
-Connection ~ 7950 2200
-Connection ~ 7950 2300
 NoConn ~ 9950 1300
 Wire Wire Line
 	7950 2400 8950 2400
-Connection ~ 7950 2400
 $Comp
 L INDUCTOR_SMALL L1
@@
 Wire Wire Line
 	6350 4300 7000 4300
-Wire Wire Line
-	7950 1700 7950 2400
-Connection ~ 7950 1800
 $Comp
 L C C18
@@
 Text Notes 9200 5400 0    60   ~ 0
 I2C Level Translator
+Connection ~ 7950 2200
+Connection ~ 7950 2400
+Connection ~ 7950 2300
+Connection ~ 7950 2100
+Connection ~ 7950 1900
+Wire Wire Line
+	7950 1700 7950 2400
+Connection ~ 7950 2000
+Connection ~ 7950 1800
 $EndSCHEMATC

Commit message: First version sent to CM for review (Screaming Circuits)
Parts:
- C13, C16, C17, C19: PN (none) -> X5R/X7R, 6.3V
- C14: PN (none) -> X5R/X7R, 16V
- C18: PN (none) -> X5R/X7R, 50V
Changed lines of the file:
@@
 F 2 "Capacitors_SMD:C_0603" H 6388 7100 30  0001 C CNN
 F 3 "" H 6350 7250 60  0000 C CNN
+F 4 "X5R/X7R, 6.3V " H 6350 7250 60  0001 C CNN "PN"
 	1    6350 7250
 	1    0    0    -1
@@
 F 2 "Capacitors_SMD:C_0603" H 6688 7100 30  0001 C CNN
 F 3 "" H 6650 7250 60  0000 C CNN
+F 4 "X5R/X7R, 16V " H 6650 7250 60  0001 C CNN "PN"
 	1    6650 7250
 	1    0    0    -1
@@
 F 2 "Capacitors_SMD:C_0603" H 5188 4650 30  0001 C CNN
 F 3 "" H 5150 4800 60  0000 C CNN
+F 4 "X5R/X7R, 6.3V " H 5150 4800 60  0001 C CNN "PN"
 	1    5150 4800
 	1    0    0    -1
@@
 F 2 "Capacitors_SMD:C_0603" H 7538 4500 30  0001 C CNN
 F 3 "" H 7500 4650 60  0000 C CNN
+F 4 "X5R/X7R, 6.3V " H 7500 4650 60  0001 C CNN "PN"
 	1    7500 4650
 	1    0    0    -1
@@
 F 2 "Capacitors_SMD:C_0603" H 4888 4650 30  0001 C CNN
 F 3 "" H 4850 4800 60  0000 C CNN
+F 4 "X5R/X7R, 50V " H 4850 4800 60  0001 C CNN "PN"
 	1    4850 4800
 	1    0    0    -1
@@
 F 2 "Capacitors_SMD:C_0603" H 7888 4500 30  0001 C CNN
 F 3 "" H 7850 4650 60  0000 C CNN
+F 4 "X5R/X7R, 6.3V " H 7850 4650 60  0001 C CNN "PN"
 	1    7850 4650
 	1    0    0    -1

Commit message: Update sch with Mfg and PN fields, added Screaming Circuits to silk.
Parts:
- C13, C17, C19: Mfg (none) -> Samsung; PN X5R/X7R, 6.3V -> CL10B475KQ8NQNC; Spec (none) -> X5R/X7R, 6.3V
- C14: Mfg (none) -> Samsung; PN X5R/X7R, 16V -> CL10B104KB8SFNC; Spec (none) -> X5R/X7R, 16V
- C16: Mfg (none) -> Samsung; PN X5R/X7R, 6.3V -> CL10A106MQ8NNNC; Spec (none) -> X5R/X7R, 6.3V
- C18: value 100nF -> 0.1uF; Mfg (none) -> Samsung; PN X5R/X7R, 50V -> CL10B104KB8SFNC; Spec (none) -> X5R/X7R, 50V
- D2, D69, D70, D71, D72, D73, D74, D75: Mfg (none) -> Diodes Incorporated
- L1: Mfg (none) -> Laird
- R1: Mfg (none) -> Yageo; PN (none) -> RC0603FR-0710KL
- R10: Mfg (none) -> Yageo; PN (none) -> RC0603FR-07100KL
- R11: Mfg (none) -> Yageo; PN (none) -> RC0603FR-071ML
- R9: Mfg (none) -> Yageo; PN (none) -> RC0603FR-07200KL
- SW5: Mfg (none) -> TE Connectivity Alcoswitch
- U2: Mfg (none) -> ams AG
- U6: Mfg (none) -> TI
- U7: Mfg (none) -> ON Semiconductor
Changed lines of the file:
@@
 F 2 "Resistors_SMD:R_0603" V 10130 2400 30  0001 C CNN
 F 3 "" H 10200 2400 30  0000 C CNN
+F 4 "Yageo" V 10200 2400 60  0001 C CNN "Mfg"
+F 5 "RC0603FR-0710KL" V 10200 2400 60  0001 C CNN "PN"
 	1    10200 2400
 	0    1    1    0
@@
 F 2 "Capacitors_SMD:C_0603" H 6388 7100 30  0001 C CNN
 F 3 "" H 6350 7250 60  0000 C CNN
-F 4 "X5R/X7R, 6.3V " H 6350 7250 60  0001 C CNN "PN"
+F 4 "X5R/X7R, 6.3V " H 6350 7250 60  0001 C CNN "Spec"
+F 5 "Samsung" H 6350 7250 60  0001 C CNN "Mfg"
+F 6 "CL10B475KQ8NQNC" H 6350 7250 60  0001 C CNN "PN"
 	1    6350 7250
 	1    0    0    -1
@@
 F 2 "Capacitors_SMD:C_0603" H 6688 7100 30  0001 C CNN
 F 3 "" H 6650 7250 60  0000 C CNN
-F 4 "X5R/X7R, 16V " H 6650 7250 60  0001 C CNN "PN"
+F 4 "X5R/X7R, 16V " H 6650 7250 60  0001 C CNN "Spec"
+F 5 "Samsung" H 6650 7250 60  0001 C CNN "Mfg"
+F 6 "CL10B104KB8SFNC" H 6650 7250 60  0001 C CNN "PN"
 	1    6650 7250
 	1    0    0    -1
@@
 F 4 "AS1115-BSST" H 9150 1100 60  0001 C CNN "PN"
 F 5 "2.11" H 9150 1100 60  0001 C CNN "Kcost"
+F 6 "ams AG" H 9150 1100 60  0001 C CNN "Mfg"
 	1    9150 1100
 	1    0    0    -1
@@
 F 4 "0.03" H 6600 1150 60  0001 C CNN "Kcost"
 F 5 "1N4148W-7-F" H 6600 1150 60  0001 C CNN "PN"
+F 6 "Diodes Incorporated" H 6600 1150 60  0001 C CNN "Mfg"
 	1    6600 1150
 	-1   0    0    1
@@
 F 4 "1-1825058-9" H 7550 2050 60  0001 C CNN "PN"
 F 5 "0.586" H 7550 2050 60  0001 C CNN "Kcost"
+F 6 "TE Connectivity Alcoswitch" H 7550 2050 60  0001 C CNN "Mfg"
 	1    7550 2050
 	-1   0    0    -1
@@
 F 4 "TYS30124R7M-10" H 5600 4850 60  0001 C CNN "PN"
 F 5 "0.18" H 5600 4850 60  0001 C CNN "Kcost"
+F 6 "Laird" H 5600 4850 60  0001 C CNN "Mfg"
 	1    5600 4850
 	0    -1   -1   0
@@
 F 4 "TPS61070DDCR" H 6000 5100 60  0001 C CNN "PN"
 F 5 "0.50" H 6000 5100 60  0001 C CNN "Kcost"
+F 6 "TI" H 6000 5100 60  0001 C CNN "Mfg"
 	1    6000 5100
 	0    -1   -1   0
@@
 F 2 "Resistors_SMD:R_0603" V 7080 4300 30  0001 C CNN
 F 3 "" H 7150 4300 30  0000 C CNN
+F 4 "Yageo" V 7150 4300 60  0001 C CNN "Mfg"
+F 5 "RC0603FR-071ML" V 7150 4300 60  0001 C CNN "PN"
 	1    7150 4300
 	0    1    1    0
@@
 F 2 "Resistors_SMD:R_0603" V 6730 4650 30  0001 C CNN
 F 3 "" H 6800 4650 30  0000 C CNN
+F 4 "Yageo" V 6800 4650 60  0001 C CNN "Mfg"
+F 5 "RC0603FR-07200KL" V 6800 4650 60  0001 C CNN "PN"
 	1    6800 4650
 	-1   0    0    1
@@
 F 2 "Resistors_SMD:R_0603" V 6730 5550 30  0001 C CNN
 F 3 "" H 6800 5550 30  0000 C CNN
+F 4 "Yageo" V 6800 5550 60  0001 C CNN "Mfg"
+F 5 "RC0603FR-07100KL" V 6800 5550 60  0001 C CNN "PN"
 	1    6800 5550
 	-1   0    0    1
@@
 F 2 "Capacitors_SMD:C_0603" H 5188 4650 30  0001 C CNN
 F 3 "" H 5150 4800 60  0000 C CNN
-F 4 "X5R/X7R, 6.3V " H 5150 4800 60  0001 C CNN "PN"
+F 4 "X5R/X7R, 6.3V " H 5150 4800 60  0001 C CNN "Spec"
+F 5 "Samsung" H 5150 4800 60  0001 C CNN "Mfg"
+F 6 "CL10A106MQ8NNNC" H 5150 4800 60  0001 C CNN "PN"
 	1    5150 4800
 	1    0    0    -1
@@
 F 2 "Capacitors_SMD:C_0603" H 7538 4500 30  0001 C CNN
 F 3 "" H 7500 4650 60  0000 C CNN
-F 4 "X5R/X7R, 6.3V " H 7500 4650 60  0001 C CNN "PN"
+F 4 "X5R/X7R, 6.3V " H 7500 4650 60  0001 C CNN "Spec"
+F 5 "Samsung" H 7500 4650 60  0001 C CNN "Mfg"
+F 6 "CL10B475KQ8NQNC" H 7500 4650 60  0001 C CNN "PN"
 	1    7500 4650
 	1    0    0    -1
@@
 P 4850 4800
 F 0 "C18" H 4875 4900 50  0000 L CNN
-F 1 "100nF" H 4875 4700 50  0000 L CNN
+F 1 "0.1uF" H 4875 4700 50  0000 L CNN
 F 2 "Capacitors_SMD:C_0603" H 4888 4650 30  0001 C CNN
 F 3 "" H 4850 4800 60  0000 C CNN
-F 4 "X5R/X7R, 50V " H 4850 4800 60  0001 C CNN "PN"
+F 4 "X5R/X7R, 50V " H 4850 4800 60  0001 C CNN "Spec"
+F 5 "Samsung" H 4850 4800 60  0001 C CNN "Mfg"
+F 6 "CL10B104KB8SFNC" H 4850 4800 60  0001 C CNN "PN"
 	1    4850 4800
 	1    0    0    -1
@@
 F 2 "Capacitors_SMD:C_0603" H 7888 4500 30  0001 C CNN
 F 3 "" H 7850 4650 60  0000 C CNN
-F 4 "X5R/X7R, 6.3V " H 7850 4650 60  0001 C CNN "PN"
+F 4 "X5R/X7R, 6.3V " H 7850 4650 60  0001 C CNN "Spec"
+F 5 "Samsung" H 7850 4650 60  0001 C CNN "Mfg"
+F 6 "CL10B475KQ8NQNC" H 7850 4650 60  0001 C CNN "PN"
 	1    7850 4650
 	1    0    0    -1
@@
 F 4 "0.03" H 6600 1400 60  0001 C CNN "Kcost"
 F 5 "1N4148W-7-F" H 6600 1400 60  0001 C CNN "PN"
+F 6 "Diodes Incorporated" H 6600 1400 60  0001 C CNN "Mfg"
 	1    6600 1400
 	-1   0    0    1
@@
 F 4 "0.03" H 6600 1650 60  0001 C CNN "Kcost"
 F 5 "1N4148W-7-F" H 6600 1650 60  0001 C CNN "PN"
+F 6 "Diodes Incorporated" H 6600 1650 60  0001 C CNN "Mfg"
 	1    6600 1650
 	-1   0    0    1
@@
 F 4 "0.03" H 6600 1900 60  0001 C CNN "Kcost"
 F 5 "1N4148W-7-F" H 6600 1900 60  0001 C CNN "PN"
+F 6 "Diodes Incorporated" H 6600 1900 60  0001 C CNN "Mfg"
 	1    6600 1900
 	-1   0    0    1
@@
 F 4 "0.03" H 6600 2150 60  0001 C CNN "Kcost"
 F 5 "1N4148W-7-F" H 6600 2150 60  0001 C CNN "PN"
+F 6 "Diodes Incorporated" H 6600 2150 60  0001 C CNN "Mfg"
 	1    6600 2150
 	-1   0    0    1
@@
 F 4 "0.03" H 6600 2400 60  0001 C CNN "Kcost"
 F 5 "1N4148W-7-F" H 6600 2400 60  0001 C CNN "PN"
+F 6 "Diodes Incorporated" H 6600 2400 60  0001 C CNN "Mfg"
 	1    6600 2400
 	-1   0    0    1
@@
 F 4 "0.03" H 6600 2650 60  0001 C CNN "Kcost"
 F 5 "1N4148W-7-F" H 6600 2650 60  0001 C CNN "PN"
+F 6 "Diodes Incorporated" H 6600 2650 60  0001 C CNN "Mfg"
 	1    6600 2650
 	-1   0    0    1
@@
 F 4 "0.03" H 6600 2900 60  0001 C CNN "Kcost"
 F 5 "1N4148W-7-F" H 6600 2900 60  0001 C CNN "PN"
+F 6 "Diodes Incorporated" H 6600 2900 60  0001 C CNN "Mfg"
 	1    6600 2900
 	-1   0    0    1
@@
 F 4 "0.40" H 9600 5600 60  0001 C CNN "Kcost"
 F 5 "NLSX4373" H 9600 5600 60  0001 C CNN "PN"
+F 6 "ON Semiconductor" H 9600 5600 60  0001 C CNN "Mfg"
 	1    9600 5600
 	1    0    0    -1

Commit message: Change to refactored Kicad local libraries
Parts:
- D10, D11, D12, D13, D14, D15, D16, D17, D18, D19, D20, D21, D22, D23, D24, D25, D26, D27, D28, D29, D3, D30, D31, D32, D33, D34, D35, D36, D37, D38, D39, D4, D40, D41, D42, D43, D44, D45, D46, D47, D48, D49, D5, D50, D51, D52, D53, D54, D55, D56, D57, D58, D59, D6, D60, D61, D62, D63, D64, D67, D68, D7, D8, D9: footprint w_smd_leds:Led_0603 -> Added:Led_0603
- D2, D69, D70, D71, D72, D73, D74, D75: footprint Diodes_SMD:SOD-323 -> Added:SOD-323
- L1: footprint Synapse:TYS-2 -> Added:TYS-2
- SW5: footprint Synapse:DIPSW-16 -> Added:DIPSW-16
- U2: footprint Synapse:QSOP-24 -> Added:QSOP-24
