File: LED_matrix.sch (KiCad schematic (older format))
At the start: 87 parts, among them SW5 SW_DIP_8, U2 AS1115, U6 TPS61070, U7 NLSX4373

Commit message: Fixed LED silkscreen, added logos
Parts:
- D2, D69, D70, D71, D72, D73, D74, D75: PN 1N4148W-7-F -> 1N4148WS-7-F
Changed lines of the file:
@@
 F 1 "1N4148W" H 6450 1070 50  0000 L CNN
 F 2 "Added:SOD-323" V 6600 1150 60  0001 C CNN
-F 3 "http://www.digikey.com/product-detail/en/1N4148W-7-F/1N4148W-FDITR-ND/814371" V 6600 1150 60  0001 C CNN
+F 3 "http://www.digikey.com/product-detail/en/1N4148WS-7-F/1N4148WS-FDICT-ND/815281" V 6600 1150 60  0001 C CNN
 F 4 "0.03" H 6600 1150 60  0001 C CNN "Kcost"
-F 5 "1N4148W-7-F" H 6600 1150 60  0001 C CNN "PN"
+F 5 "1N4148WS-7-F" H 6600 1150 60  0001 C CNN "PN"
 F 6 "Diodes Incorporated" H 6600 1150 60  0001 C CNN "Mfg"
 	1    6600 1150
@@
 F 1 "1N4148W" H 6450 1320 50  0000 L CNN
 F 2 "Added:SOD-323" V 6600 1400 60  0001 C CNN
-F 3 "http://www.digikey.com/product-detail/en/1N4148W-7-F/1N4148W-FDITR-ND/814371" V 6600 1400 60  0001 C CNN
+F 3 "http://www.digikey.com/product-detail/en/1N4148WS-7-F/1N4148WS-FDICT-ND/815281" V 6600 1400 60  0001 C CNN
 F 4 "0.03" H 6600 1400 60  0001 C CNN "Kcost"
-F 5 "1N4148W-7-F" H 6600 1400 60  0001 C CNN "PN"
+F 5 "1N4148WS-7-F" H 6600 1400 60  0001 C CNN "PN"
 F 6 "Diodes Incorporated" H 6600 1400 60  0001 C CNN "Mfg"
 	1    6600 1400
@@
 F 1 "1N4148W" H 6450 1570 50  0000 L CNN
 F 2 "Added:SOD-323" V 6600 1650 60  0001 C CNN
-F 3 "http://www.digikey.com/product-detail/en/1N4148W-7-F/1N4148W-FDITR-ND/814371" V 6600 1650 60  0001 C CNN
+F 3 "http://www.digikey.com/product-detail/en/1N4148WS-7-F/1N4148WS-FDICT-ND/815281" V 6600 1650 60  0001 C CNN
 F 4 "0.03" H 6600 1650 60  0001 C CNN "Kcost"
-F 5 "1N4148W-7-F" H 6600 1650 60  0001 C CNN "PN"
+F 5 "1N4148WS-7-F" H 6600 1650 60  0001 C CNN "PN"
 F 6 "Diodes Incorporated" H 6600 1650 60  0001 C CNN "Mfg"
 	1    6600 1650
@@
 F 1 "1N4148W" H 6450 1820 50  0000 L CNN
 F 2 "Added:SOD-323" V 6600 1900 60  0001 C CNN
-F 3 "http://www.digikey.com/product-detail/en/1N4148W-7-F/1N4148W-FDITR-ND/814371" V 6600 1900 60  0001 C CNN
+F 3 "http://www.digikey.com/product-detail/en/1N4148WS-7-F/1N4148WS-FDICT-ND/815281" V 6600 1900 60  0001 C CNN
 F 4 "0.03" H 6600 1900 60  0001 C CNN "Kcost"
-F 5 "1N4148W-7-F" H 6600 1900 60  0001 C CNN "PN"
+F 5 "1N4148WS-7-F" H 6600 1900 60  0001 C CNN "PN"
 F 6 "Diodes Incorporated" H 6600 1900 60  0001 C CNN "Mfg"
 	1    6600 1900
@@
 F 1 "1N4148W" H 6450 2070 50  0000 L CNN
 F 2 "Added:SOD-323" V 6600 2150 60  0001 C CNN
-F 3 "http://www.digikey.com/product-detail/en/1N4148W-7-F/1N4148W-FDITR-ND/814371" V 6600 2150 60  0001 C CNN
+F 3 "http://www.digikey.com/product-detail/en/1N4148WS-7-F/1N4148WS-FDICT-ND/815281" V 6600 2150 60  0001 C CNN
 F 4 "0.03" H 6600 2150 60  0001 C CNN "Kcost"
-F 5 "1N4148W-7-F" H 6600 2150 60  0001 C CNN "PN"
+F 5 "1N4148WS-7-F" H 6600 2150 60  0001 C CNN "PN"
 F 6 "Diodes Incorporated" H 6600 2150 60  0001 C CNN "Mfg"
 	1    6600 2150
@@
 F 1 "1N4148W" H 6450 2320 50  0000 L CNN
 F 2 "Added:SOD-323" V 6600 2400 60  0001 C CNN
-F 3 "http://www.digikey.com/product-detail/en/1N4148W-7-F/1N4148W-FDITR-ND/814371" V 6600 2400 60  0001 C CNN
+F 3 "http://www.digikey.com/product-detail/en/1N4148WS-7-F/1N4148WS-FDICT-ND/815281" V 6600 2400 60  0001 C CNN
 F 4 "0.03" H 6600 2400 60  0001 C CNN "Kcost"
-F 5 "1N4148W-7-F" H 6600 2400 60  0001 C CNN "PN"
+F 5 "1N4148WS-7-F" H 6600 2400 60  0001 C CNN "PN"
 F 6 "Diodes Incorporated" H 6600 2400 60  0001 C CNN "Mfg"
 	1    6600 2400
@@
 F 1 "1N4148W" H 6450 2570 50  0000 L CNN
 F 2 "Added:SOD-323" V 6600 2650 60  0001 C CNN
-F 3 "http://www.digikey.com/product-detail/en/1N4148W-7-F/1N4148W-FDITR-ND/814371" V 6600 2650 60  0001 C CNN
+F 3 "http://www.digikey.com/product-detail/en/1N4148WS-7-F/1N4148WS-FDICT-ND/815281" V 6600 2650 60  0001 C CNN
 F 4 "0.03" H 6600 2650 60  0001 C CNN "Kcost"
-F 5 "1N4148W-7-F" H 6600 2650 60  0001 C CNN "PN"
+F 5 "1N4148WS-7-F" H 6600 2650 60  0001 C CNN "PN"
 F 6 "Diodes Incorporated" H 6600 2650 60  0001 C CNN "Mfg"
 	1    6600 2650
@@
 F 1 "1N4148W" H 6450 2820 50  0000 L CNN
 F 2 "Added:SOD-323" V 6600 2900 60  0001 C CNN
-F 3 "http://www.digikey.com/product-detail/en/1N4148W-7-F/1N4148W-FDITR-ND/814371" V 6600 2900 60  0001 C CNN
+F 3 "http://www.digikey.com/product-detail/en/1N4148WS-7-F/1N4148WS-FDICT-ND/815281" V 6600 2900 60  0001 C CNN
 F 4 "0.03" H 6600 2900 60  0001 C CNN "Kcost"
-F 5 "1N4148W-7-F" H 6600 2900 60  0001 C CNN "PN"
+F 5 "1N4148WS-7-F" H 6600 2900 60  0001 C CNN "PN"
 F 6 "Diodes Incorporated" H 6600 2900 60  0001 C CNN "Mfg"
 	1    6600 2900
