File: SNAP_badge.sch (KiCad schematic (older format))
At the start: 51 parts, among them P1 MicroB, P2 CONN_01X08, P3 CONN_01X08, P4 CONN_01X10, P5 CONN_01X06, P6 CONN_02X03, Q1 ZXMN2F30FHCT-ND, Q2 Si2305DS, SW1 SWITCH_DPDT, SW2 SW_PUSH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

Commit message: Change to refactored Kicad local libraries
Parts:
- BT1, BT2: footprint Synapse:BATT_2466 -> Added:BATT_2466
- D1, D65, D66: footprint w_smd_leds:Led_0603 -> Added:Led_0603
- P1: footprint Synapse:USBmicroB -> Added:USBmicroB
- SW1: footprint Synapse:SO-DPDT-6 -> Added:SO-DPDT-6
- SW2, SW3, SW4: footprint Buttons_Switches_SMD:SW_SPST_PTS645 -> Added:SW_SPST_PTS645
- U5: footprint Synapse:LGA16_3x3 -> Added:LGA16_3x3
Changed lines of the file:
@@
 LIBS:contrib
 LIBS:valves
-LIBS:sm220
-LIBS:FT230XS
-LIBS:SWITCH_DPDT
+LIBS:as111x
+LIBS:ftdi
+LIBS:nlsx4373
 LIBS:STM_MEMS
-LIBS:as111x
 LIBS:sw_dip
-LIBS:regulators
-LIBS:nlsx4373
-LIBS:test_board2-cache
+LIBS:switches
+LIBS:synapse
+LIBS:TI_buckboost
+LIBS:SNAP_badge-cache
 EELAYER 25 0
 EELAYER END
@@
 F 0 "D65" H 10600 5600 50  0000 C CNN
 F 1 "LED" H 10600 5400 50  0000 C CNN
-F 2 "w_smd_leds:Led_0603" H 10600 5500 60  0001 C CNN
+F 2 "Added:Led_0603" H 10600 5500 60  0001 C CNN
 F 3 "" H 10600 5500 60  0000 C CNN
 	1    10600 5500
@@
 F 0 "D66" H 10950 5700 50  0000 C CNN
 F 1 "LED" H 10950 5500 50  0000 C CNN
-F 2 "w_smd_leds:Led_0603" H 10950 5600 60  0001 C CNN
+F 2 "Added:Led_0603" H 10950 5600 60  0001 C CNN
 F 3 "" H 10950 5600 60  0000 C CNN
 	1    10950 5600
@@
 F 0 "SW1" H 3300 7400 70  0000 C CNN
 F 1 "SWITCH_DPDT" H 3300 6500 70  0000 C CNN
-F 2 "Synapse:SO-DPDT-6" H 3300 6950 60  0001 C CNN
+F 2 "Added:SO-DPDT-6" H 3300 6950 60  0001 C CNN
 F 3 "http://www.digikey.com/product-detail/en/JS202011SCQN/401-2002-2-ND/2094299" H 3300 6950 60  0001 C CNN
 F 4 "JS202011SCQN" H 3300 6950 60  0001 C CNN "PN"
@@
 F 0 "BT2" H 1500 5350 50  0000 L CNN
 F 1 "1.5V" H 1500 5250 50  0000 L CNN
-F 2 "Synapse:BATT_2466" V 1400 5340 60  0001 C CNN
+F 2 "Added:BATT_2466" V 1400 5340 60  0001 C CNN
 F 3 "http://www.digikey.com/product-detail/en/2466/36-2466-ND/303815" V 1400 5340 60  0001 C CNN
 F 4 ".59" H 1400 5300 60  0001 C CNN "Kcost"
@@
 F 0 "U5" H 9150 2250 60  0000 C CNN
 F 1 "LIS3DH" H 9700 1700 60  0000 C CNN
-F 2 "Synapse:LGA16_3x3" H 9650 1750 60  0001 C CNN
+F 2 "Added:LGA16_3x3" H 9650 1750 60  0001 C CNN
 F 3 "http://www.digikey.com/product-detail/en/LIS3DHTR/497-10613-1-ND/2334355" H 9650 1750 60  0001 C CNN
 F 4 "LIS3DHTR" H 9650 1750 60  0001 C CNN "PN"
@@
 F 0 "SW2" H 10200 3360 50  0000 C CNN
 F 1 "SW_PUSH" H 10050 3170 50  0000 C CNN
-F 2 "Buttons_Switches_SMD:SW_SPST_PTS645" H 10050 3250 60  0001 C CNN
+F 2 "Added:SW_SPST_PTS645" H 10050 3250 60  0001 C CNN
 F 3 "http://www.digikey.com/product-detail/en/PTS645SL50SMTR92%20LFS/CKN9088TR-ND/1279107" H 10050 3250 60  0001 C CNN
 F 4 "PTS645SL50SMTR92 LFS" H 10050 3250 60  0001 C CNN "PN"
@@
 F 0 "D1" H 7750 2700 50  0000 C CNN
 F 1 "LED" H 7750 2500 50  0000 C CNN
-F 2 "w_smd_leds:Led_0603" H 7750 2600 60  0001 C CNN
+F 2 "Added:Led_0603" H 7750 2600 60  0001 C CNN
 F 3 "" H 7750 2600 60  0000 C CNN
 	1    7750 2600
@@
 F 0 "SW3" H 10200 3660 50  0000 C CNN
 F 1 "SW_PUSH" H 10050 3470 50  0000 C CNN
-F 2 "Buttons_Switches_SMD:SW_SPST_PTS645" H 10050 3550 60  0001 C CNN
+F 2 "Added:SW_SPST_PTS645" H 10050 3550 60  0001 C CNN
 F 3 "http://www.digikey.com/product-detail/en/PTS645SL50SMTR92%20LFS/CKN9088TR-ND/1279107" H 10050 3550 60  0001 C CNN
 F 4 "PTS645SL50SMTR92 LFS" H 10050 3550 60  0001 C CNN "PN"
@@
 F 0 "SW4" H 10200 3960 50  0000 C CNN
 F 1 "SW_PUSH" H 10050 3770 50  0000 C CNN
-F 2 "Buttons_Switches_SMD:SW_SPST_PTS645" H 10050 3850 60  0001 C CNN
+F 2 "Added:SW_SPST_PTS645" H 10050 3850 60  0001 C CNN
 F 3 "http://www.digikey.com/product-detail/en/PTS645SL50SMTR92%20LFS/CKN9088TR-ND/1279107" H 10050 3850 60  0001 C CNN
 F 4 "PTS645SL50SMTR92 LFS" H 10050 3850 60  0001 C CNN "PN"
@@
 F 0 "P1" H 6625 5375 50  0000 C CNN
 F 1 "MicroB" H 6300 5700 50  0000 C CNN
-F 2 "Synapse:USBmicroB" V 6250 5400 60  0001 C CNN
+F 2 "Added:USBmicroB" V 6250 5400 60  0001 C CNN
 F 3 "http://www.digikey.com/product-detail/en/10118194-0001LF/609-4618-2-ND/2785389" V 6250 5400 60  0001 C CNN
 F 4 "0.20" H 6300 5500 60  0001 C CNN "Kcost"
@@
 F 0 "BT1" H 1500 5700 50  0000 L CNN
 F 1 "1.5V" H 1500 5600 50  0000 L CNN
-F 2 "Synapse:BATT_2466" V 1400 5690 60  0001 C CNN
+F 2 "Added:BATT_2466" V 1400 5690 60  0001 C CNN
 F 3 "http://www.digikey.com/product-detail/en/2466/36-2466-ND/303815" V 1400 5690 60  0001 C CNN
 F 4 ".59" H 1400 5650 60  0001 C CNN "Kcost"

Commit message: Fixed LED silkscreen, added logos
Parts:
- P2, P3: Kcost .64 -> .36; Mfg FCI -> Sullins; PN FCI 75915-308LF -> PPPC081LFBN-RC
- P4: Kcost .78 -> .36; Mfg FCI -> Sullins; PN FCI 75915-310LF -> PPPC101LFBN-RC
- P5: Kcost .49 -> .29; Mfg FCI -> Sullins; PN FCI 75915-306LF -> PPPC061LFBN-RC
Changed lines of the file:
@@
 F 1 "CONN_01X08" V 1400 2750 50  0000 C CNN
 F 2 "Socket_Strips:Socket_Strip_Straight_1x08" H 1300 2750 60  0001 C CNN
-F 3 "http://www.digikey.com/product-detail/en/75915-308LF/609-3559-ND/1523940" H 1300 2750 60  0001 C CNN
-F 4 "FCI 75915-308LF" H 1300 2750 60  0001 C CNN "PN"
-F 5 ".64" H 1300 2750 60  0001 C CNN "Kcost"
-F 6 "FCI" H 1300 2750 60  0001 C CNN "Mfg"
+F 3 "http://www.digikey.com/product-detail/en/PPPC081LFBN-RC/S7041-ND/810180" H 1300 2750 60  0001 C CNN
+F 4 "PPPC081LFBN-RC" H 1300 2750 60  0001 C CNN "PN"
+F 5 ".36" H 1300 2750 60  0001 C CNN "Kcost"
+F 6 "Sullins" H 1300 2750 60  0001 C CNN "Mfg"
 	1    1300 2750
 	1    0    0    -1
@@
 F 1 "CONN_01X08" V 2550 3500 50  0000 C CNN
 F 2 "Socket_Strips:Socket_Strip_Straight_1x08" H 2450 3500 60  0001 C CNN
-F 3 "http://www.digikey.com/product-detail/en/75915-308LF/609-3559-ND/1523940" H 2450 3500 60  0001 C CNN
-F 4 "FCI 75915-308LF" H 2450 3500 60  0001 C CNN "PN"
-F 5 ".64" H 2450 3500 60  0001 C CNN "Kcost"
-F 6 "FCI" H 2450 3500 60  0001 C CNN "Mfg"
+F 3 "http://www.digikey.com/product-detail/en/PPPC081LFBN-RC/S7041-ND/810180" H 2450 3500 60  0001 C CNN
+F 4 "PPPC081LFBN-RC" H 2450 3500 60  0001 C CNN "PN"
+F 5 ".36" H 2450 3500 60  0001 C CNN "Kcost"
+F 6 "Sullins" H 2450 3500 60  0001 C CNN "Mfg"
 	1    2450 3500
 	1    0    0    -1
@@
 F 1 "CONN_01X10" V 2550 2400 50  0000 C CNN
 F 2 "Socket_Strips:Socket_Strip_Straight_1x10" H 2450 2400 60  0001 C CNN
-F 3 "http://www.digikey.com/product-detail/en/75915-310LF/609-3550-ND/1524287" H 2450 2400 60  0001 C CNN
-F 4 ".78" H 2450 2400 60  0001 C CNN "Kcost"
-F 5 "FCI 75915-310LF" H 2450 2400 60  0001 C CNN "PN"
-F 6 "FCI" H 2450 2400 60  0001 C CNN "Mfg"
+F 3 "http://www.digikey.com/product-detail/en/PPPC101LFBN-RC/S7043-ND/810182" H 2450 2400 60  0001 C CNN
+F 4 ".36" H 2450 2400 60  0001 C CNN "Kcost"
+F 5 "PPPC101LFBN-RC" H 2450 2400 60  0001 C CNN "PN"
+F 6 "Sullins" H 2450 2400 60  0001 C CNN "Mfg"
 	1    2450 2400
 	1    0    0    -1
@@
 F 1 "CONN_01X06" V 1400 3600 50  0000 C CNN
 F 2 "Socket_Strips:Socket_Strip_Straight_1x06" H 1300 3600 60  0001 C CNN
-F 3 "http://www.digikey.com/product-detail/en/75915-306LF/609-3558-ND/1523584" H 1300 3600 60  0001 C CNN
-F 4 ".49" H 1300 3600 60  0001 C CNN "Kcost"
-F 5 "FCI 75915-306LF" H 1300 3600 60  0001 C CNN "PN"
-F 6 "FCI" H 1300 3600 60  0001 C CNN "Mfg"
+F 3 "http://www.digikey.com/product-detail/en/PPPC061LFBN-RC/S7039-ND/810178" H 1300 3600 60  0001 C CNN
+F 4 ".29" H 1300 3600 60  0001 C CNN "Kcost"
+F 5 "PPPC061LFBN-RC" H 1300 3600 60  0001 C CNN "PN"
+F 6 "Sullins" H 1300 3600 60  0001 C CNN "Mfg"
 	1    1300 3600
 	1    0    0    -1
